File: board/board.kicad_pcb (KiCad board)
At the start: 4 copper layers, 260.6 x 185.6 mm, 114 parts, among them J1 Conn_01x05_Pin, J10 VGA, J2 KEYBOARD, J3 AdaFruit 4090 USB-C BOB, J4 MOUSE, J5 OBVID_JTAG_BYPASS, J6 COMPOSITE, J7 STEREO_OUT, J8 CF Card, J9 FTDI serial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

Commit message: JTAG bypass, GLUE A18, OBVID pins
Fix up JTAG bypass again
Switch GLUE A6 to GLUE A18
Clean up some OBVID pins
Connections:
- U12 pad 81: A6 -> A18
Routing:
- net A18: track 454.3 -> 480.7 mm, vias 7 -> 8
- net A6: track 429.7 -> 404.2 mm, vias 7 -> 6
