File: board/board.kicad_sch (KiCad schematic)
At the start: 0 parts

Commit message: change OBVID to VIDEO
Other:
- sheet APP_ENGINE renamed ENGINE
- sheet ONBOARDVID renamed VIDEO
Changed lines of the file:
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@@
 			(color 0 0 0 0.0000)
 		)
-		(property "Sheetname" "ONBOARDVID"
+		(property "Sheetname" "VIDEO"
 			(at 88.9 100.8884 0)
 			(effects
@@
 			(color 0 0 0 0.0000)
 		)
-		(property "Sheetname" "APP_ENGINE"
+		(property "Sheetname" "ENGINE"
 			(at 152.4 100.8884 0)
 			(effects
