File: board/board.kicad_sch (KiCad schematic)
At the start: 0 parts

Commit message: update parts I've added
Other:
- sheet VIDEO renamed TIMING
- added sheet VIDEO1 (composite.kicad_sch)
Changed lines of the file:
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@@
 			(color 0 0 0 0.0000)
 		)
-		(property "Sheetname" "VIDEO"
+		(property "Sheetname" "TIMING"
 			(at 88.9 100.8884 0)
 			(effects
@@
 				)
 			)
+		)
+	)
+	(sheet
+		(at 152.4 138.43)
+		(size 40 20)
+		(exclude_from_sim no)
+		(in_bom yes)
+		(on_board yes)
+		(dnp no)
+		(fields_autoplaced yes)
+		(stroke
+			(width 0.1524)
+			(type solid)
+		)
+		(fill
+			(color 0 0 0 0.0000)
+		)
+		(property "Sheetname" "VIDEO1"
+			(at 152.4 137.7184 0)
+			(effects
+				(font
+					(size 1.27 1.27)
+				)
+				(justify left bottom)
+			)
+		)
+		(property "Sheetfile" "composite.kicad_sch"
+			(at 152.4 165.6846 0)
+			(effects
+				(font
+					(size 1.27 1.27)
+				)
+				(justify left top)
+			)
+		)
+		(instances
+			(project "board"
+				(path "/afefa398-9f39-4b22-97f8-dae9b102df0d"
+					(page "13")
+				)
+			)

Commit message: checkpoint
Other:
- sheet POWER_CLOCK renamed POWER_CLOCK_RESET
Changed lines of the file:
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@@
 			(color 0 0 0 0.0000)
 		)
-		(property "Sheetname" "POWER_CLOCK"
+		(property "Sheetname" "POWER_CLOCK_RESET"
 			(at 25.4 24.6884 0)
 			(effects

Commit message: checkpoint
Other:
- removed sheet VIDEO1
- added sheet PORTS (glue.kicad_sch)
Changed lines of the file:
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@@
 	)
 	(sheet
-		(at 152.4 138.43)
+		(at 215.9 25.4)
 		(size 40 20)
 		(exclude_from_sim no)
@@
 			(color 0 0 0 0.0000)
 		)
-		(property "Sheetname" "VIDEO1"
-			(at 152.4 137.7184 0)
+		(property "Sheetname" "PORTS"
+			(at 215.9 24.6884 0)
 			(effects
 				(font
@@
 			)
 		)
-		(property "Sheetfile" "composite.kicad_sch"
-			(at 152.4 165.6846 0)
+		(property "Sheetfile" "glue.kicad_sch"
+			(at 215.9 50.1146 0)
 			(effects
 				(font
@@
 			(project "board"
 				(path "/afefa398-9f39-4b22-97f8-dae9b102df0d"
-					(page "13")
+					(page "7")
 				)
 			)

Commit message: capture ENGINE in schematic; fix couple of shorts
Other:
- sheet PORTS: file glue.kicad_sch -> ports.kicad_sch
Changed lines of the file:
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@@
 			)
 		)
-		(property "Sheetfile" "glue.kicad_sch"
+		(property "Sheetfile" "ports.kicad_sch"
 			(at 215.9 50.1146 0)
 			(effects

Commit message: capture TIMING; add PLCC44 ATF1504; a few fixes
Changed lines of the file:
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@@
 		(on_board yes)
 		(dnp no)
-		(fields_autoplaced yes)
 		(stroke
 			(width 0.1524)
@@
 		)
 		(property "Sheetfile" "composite.kicad_sch"
-			(at 88.9 128.8546 0)
+			(at 88.9 122.682 0)
 			(effects
 				(font

Commit message: checkpoint CPLDs
Other:
- added sheet COMPOSITOR (compositor.kicad_sch)
- added sheet PIXEL (pixel.kicad_sch)
Changed lines of the file:
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@@
+	)
+	(sheet
+		(at 215.9 101.6)
+		(size 40 20)
+		(exclude_from_sim no)
+		(in_bom yes)
+		(on_board yes)
+		(dnp no)
+		(fields_autoplaced yes)
+		(stroke
+			(width 0.1524)
+			(type solid)
+		)
+		(fill
+			(color 0 0 0 0.0000)
+		)
+		(property "Sheetname" "PIXEL"
+			(at 215.9 100.8884 0)
+			(effects
+				(font
+					(size 1.27 1.27)
+				)
+				(justify left bottom)
+			)
+		)
+		(property "Sheetfile" "pixel.kicad_sch"
+			(at 215.9 125.0446 0)
+			(effects
+				(font
+					(size 1.27 1.27)
+				)
+				(justify left top)
+			)
+		)
+		(instances
+			(project "board"
+				(path "/afefa398-9f39-4b22-97f8-dae9b102df0d"
+					(page "13")
+				)
+			)
+		)
 	)
 	(sheet
@@
 				)
 			)
+		)
+	)
+	(sheet
+		(at 215.9 138.43)
+		(size 40 20)
+		(exclude_from_sim no)
+		(in_bom yes)
+		(on_board yes)
+		(dnp no)
+		(fields_autoplaced yes)
+		(stroke
+			(width 0.1524)
+			(type solid)
+		)
+		(fill
+			(color 0 0 0 0.0000)
+		)
+		(property "Sheetname" "COMPOSITOR"
+			(at 215.9 137.7184 0)
+			(effects
+				(font
+					(size 1.27 1.27)
+				)
+				(justify left bottom)
+			)
+		)
+		(property "Sheetfile" "compositor.kicad_sch"
+			(at 215.9 161.8746 0)
+			(effects
+				(font
+					(size 1.27 1.27)
+				)
+				(justify left top)
+			)
+		)
+		(instances
+			(project "board"
+				(path "/afefa398-9f39-4b22-97f8-dae9b102df0d"
+					(page "14")
+				)
+			)
