File: board/board.kicad_sch (KiCad schematic)
At the start: 0 parts

Commit message: rename AUDIO sheet to AUDIO_DAC (debug-led.kicad_sch -> audio-dac.kicad_sch)
Co-Authored-By: Claude Fable 5.1 <noreply@anthropic.com>
Claude-Session: https://claude.ai/code/session_01NsFH8WNb3Tja14xUfwuyqj
Other:
- sheet AUDIO renamed AUDIO_DAC
- sheet AUDIO_DAC: file debug-led.kicad_sch -> audio-dac.kicad_sch
Changed lines of the file:
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@@
 			(color 0 0 0 0.0000)
 		)
-		(property "Sheetname" "AUDIO"
+		(property "Sheetname" "AUDIO_DAC"
 			(at 152.4 62.7884 0)
 			(effects
@@
 			)
 		)
-		(property "Sheetfile" "debug-led.kicad_sch"
+		(property "Sheetfile" "audio-dac.kicad_sch"
 			(at 152.4 88.2146 0)
 			(effects
