File: board/board.kicad_sch (KiCad schematic)
At the start: 0 parts

Commit message: add debug header
Other:
- removed sheet TESTPOINTS
Changed lines of the file:
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@@
+	)
+	(sheet
+		(at 152.4 138.43)
+		(size 40 20)
+		(exclude_from_sim no)
+		(in_bom yes)
+		(on_board yes)
+		(dnp no)
+		(fields_autoplaced yes)
+		(stroke
+			(width 0.1524)
+			(type solid)
+		)
+		(fill
+			(color 0 0 0 0.0000)
+		)
+		(property "Sheetname" "DEBUG_HEADER"
+			(at 152.4 137.7184 0)
+			(effects
+				(font
+					(size 1.27 1.27)
+				)
+				(justify left bottom)
+			)
+		)
+		(property "Sheetfile" "debug-header.kicad_sch"
+			(at 152.4 161.8746 0)
+			(effects
+				(font
+					(size 1.27 1.27)
+				)
+				(justify left top)
+			)
+		)
+		(instances
+			(project "board"
+				(path "/afefa398-9f39-4b22-97f8-dae9b102df0d"
+					(page "16")
+				)
+			)
+		)
 	)
 	(sheet
@@
 				(path "/afefa398-9f39-4b22-97f8-dae9b102df0d"
 					(page "10")
-				)
-			)
-		)
-	)
-	(sheet
-		(at 25.4 138.43)
-		(size 40.64 20.32)
-		(exclude_from_sim no)
-		(in_bom yes)
-		(on_board yes)
-		(dnp no)
-		(fields_autoplaced yes)
-		(stroke
-			(width 0.1524)
-			(type solid)
-		)
-		(fill
-			(color 0 0 0 0.0000)
-		)
-		(property "Sheetname" "TESTPOINTS"
-			(at 25.4 137.7184 0)
-			(effects
-				(font
-					(size 1.27 1.27)
-				)
-				(justify left bottom)
-			)
-		)
-		(property "Sheetfile" "test-points.kicad_sch"
-			(at 25.4 159.3346 0)
-			(effects
-				(font
-					(size 1.27 1.27)
-				)
-				(justify left top)
-			)
-		)
-		(instances
-			(project "board"
-				(path "/afefa398-9f39-4b22-97f8-dae9b102df0d"
-					(page "11")
 				)
 			)
@@
 	)
 	(embedded_fonts no)
-	(sheet
-		(at 152.4 138.43)
-		(size 40 20)
-		(exclude_from_sim no)
-		(in_bom yes)
-		(on_board yes)
-		(dnp no)
-		(fields_autoplaced yes)
-		(stroke
-			(width 0.1524)
-			(type solid)
-		)
-		(fill
-			(color 0 0 0 0.0000)
-		)
-		(property "Sheetname" "DEBUG_HEADER"
-			(at 152.4 137.7184 0)
-			(effects
-				(font
-					(size 1.27 1.27)
-				)
-				(justify left bottom)
-			)
-		)
-		(property "Sheetfile" "debug-header.kicad_sch"
-			(at 152.4 161.8746 0)
-			(effects
-				(font
-					(size 1.27 1.27)
-				)
-				(justify left top)
-			)
-		)
-		(instances
-			(project "board"
-				(path "/afefa398-9f39-4b22-97f8-dae9b102df0d"
-					(page "16")
-				)
-			)
-		)
-	)
 )
