File: board/test-points.kicad_sch (KiCad schematic)
At the start: 15 parts

Commit message: CPUCLK -> SYSCLK
Connections:
- net CPUCLK renamed SYSCLK
Changed lines of the file:
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@@
 		)
 	)
-	(global_label "CPUCLK"
+	(global_label "SYSCLK"
 		(shape input)
 		(at 60.96 30.48 180)
