File: board/compact-flash.kicad_sch (KiCad schematic)
At the start: 1 part, among them J8 CF Card

Commit message: capture ENGINE in schematic; fix couple of shorts
Parts:
- renumbered J8 to J7
Changed lines of the file:
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@@
 		(dnp no)
 		(fields_autoplaced yes)
-		(property "Reference" "#PWR061"
+		(property "Reference" "#PWR0144"
 			(at 181.61 88.9 0)
 			(effects
@@
 			(project "board"
 				(path "/afefa398-9f39-4b22-97f8-dae9b102df0d/4a375e65-a69e-4a1a-b605-646ac9dfc1ea"
-					(reference "#PWR061")
+					(reference "#PWR0144")
 					(unit 1)
 				)
@@
 		(dnp no)
 		(fields_autoplaced yes)
-		(property "Reference" "J8"
+		(property "Reference" "J7"
 			(at 143.51 55.88 0)
 			(effects
@@
 			(project "board"
 				(path "/afefa398-9f39-4b22-97f8-dae9b102df0d/4a375e65-a69e-4a1a-b605-646ac9dfc1ea"
-					(reference "J8")
+					(reference "J7")
 					(unit 1)
 				)
@@
 		(dnp no)
 		(fields_autoplaced yes)
-		(property "Reference" "#PWR070"
+		(property "Reference" "#PWR0143"
 			(at 170.18 134.62 0)
 			(effects
@@
 			(project "board"
 				(path "/afefa398-9f39-4b22-97f8-dae9b102df0d/4a375e65-a69e-4a1a-b605-646ac9dfc1ea"
-					(reference "#PWR070")
+					(reference "#PWR0143")
 					(unit 1)
 				)
@@
 		(dnp no)
 		(fields_autoplaced yes)
-		(property "Reference" "#PWR069"
+		(property "Reference" "#PWR0142"
 			(at 116.84 111.76 0)
 			(effects
@@
 			(project "board"
 				(path "/afefa398-9f39-4b22-97f8-dae9b102df0d/4a375e65-a69e-4a1a-b605-646ac9dfc1ea"
-					(reference "#PWR069")
+					(reference "#PWR0142")
 					(unit 1)
 				)
@@
 		(dnp no)
 		(fields_autoplaced yes)
-		(property "Reference" "#PWR075"
+		(property "Reference" "#PWR0141"
 			(at 113.03 82.55 0)
 			(effects
@@
 			(project "board"
 				(path "/afefa398-9f39-4b22-97f8-dae9b102df0d/4a375e65-a69e-4a1a-b605-646ac9dfc1ea"
-					(reference "#PWR075")
+					(reference "#PWR0141")
 					(unit 1)
 				)
