File: board/cpu.kicad_sch (KiCad schematic)
At the start: 5 parts, among them U1 MC68000P

Commit message: update parts I've added
Parts:
- added R10, R11, R13, R17, R18, R24, R27, R28, R29: 10K, Resistor_THT:R_Axial_DIN0207_L6.3mm_D2.5mm_P10.16mm_Horizontal, symbol Device:R
- added R8: 4.7K, Resistor_THT:R_Axial_DIN0207_L6.3mm_D2.5mm_P10.16mm_Horizontal, symbol Device:R
- R3, R4: value 100K -> 10K
- U1: value MC68000P -> MC68000
Connections:
- net FC1 is gone; now on net FC0: U1.27 (FC1)
- net ~{AS} is gone; now on net R/~{W}: U1.6 (~{AS})
- net +5V: now also R10.1, R11.1, R13.1, R17.1, R18.1, R24.1, R27.1, R28.1, R29.1, R8.1
- net FC0: now also R24.2, R27.2
- net FC2: now also R28.2
- net R/~{W}: now also R11.2, R13.2
- net ~{HALT}: now also R8.2
- net ~{LDS}: now also R18.2
- net ~{RESET}: now also R10.2
- net ~{UDS}: now also R17.2
- net ~{VPA}: now also R29.2
Other:
- moved on the sheet: R3, R4

Commit message: checkpoint
Parts:
- removed R10: 10K, Resistor_THT:R_Axial_DIN0207_L6.3mm_D2.5mm_P10.16mm_Horizontal, symbol Device:R
Changed lines of the file:
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@@
-	)
-	(junction
-		(at 113.03 135.89)
-		(diameter 0)
-		(color 0 0 0 0)
 	)
 	(junction
@@
 	)
 	(junction
-		(at 102.87 116.84)
-		(diameter 0)
-		(color 0 0 0 0)
-	)
-	(junction
 		(at 111.76 26.67)
 		(diameter 0)
@@
 	(wire
 		(pts
-			(xy 102.87 114.3) (xy 102.87 116.84)
+			(xy 102.87 114.3) (xy 102.87 119.38)
 		)
 		(stroke
@@
 	(wire
 		(pts
-			(xy 113.03 127) (xy 113.03 135.89)
-		)
-		(stroke
-			(width 0)
-			(type default)
-		)
-	)
-	(wire
-		(pts
 			(xy 127 91.44) (xy 139.7 91.44)
 		)
@@
 	(wire
 		(pts
-			(xy 96.52 135.89) (xy 113.03 135.89)
+			(xy 96.52 135.89) (xy 143.51 135.89)
 		)
 		(stroke
@@
 	(wire
 		(pts
-			(xy 102.87 116.84) (xy 113.03 116.84)
-		)
-		(stroke
-			(width 0)
-			(type default)
-		)
-	)
-	(wire
-		(pts
 			(xy 139.7 80.01) (xy 143.51 80.01)
 		)
@@
 	(wire
 		(pts
-			(xy 102.87 116.84) (xy 102.87 119.38)
-		)
-		(stroke
-			(width 0)
-			(type default)
-		)
-	)
-	(wire
-		(pts
 			(xy 124.46 91.44) (xy 127 91.44)
 		)
@@
 	(wire
 		(pts
-			(xy 113.03 135.89) (xy 143.51 135.89)
-		)
-		(stroke
-			(width 0)
-			(type default)
-		)
-	)
-	(wire
-		(pts
 			(xy 173.99 92.71) (xy 184.15 92.71)
 		)
@@
 		(pts
 			(xy 107.95 97.79) (xy 107.95 100.33)
-		)
-		(stroke
-			(width 0)
-			(type default)
-		)
-	)
-	(wire
-		(pts
-			(xy 113.03 116.84) (xy 113.03 119.38)
 		)
 		(stroke
@@
 					(unit 1)
 				)
-			)
-		)
-	)
-	(symbol
-		(lib_id "Device:R")
-		(at 113.03 123.19 0)
-		(unit 1)
-		(exclude_from_sim no)
-		(in_bom yes)
-		(on_board yes)
-		(dnp no)
-		(fields_autoplaced yes)
-		(property "Reference" "R10"
-			(at 115.57 121.9199 0)
-			(effects
-				(font
-					(size 1.27 1.27)
-				)
-				(justify left)
-			)
-		)
-		(property "Value" "10K"
-			(at 115.57 124.4599 0)
-			(effects
-				(font
-					(size 1.27 1.27)
-				)
-				(justify left)
-			)
-		)
-		(property "Footprint" "Resistor_THT:R_Axial_DIN0207_L6.3mm_D2.5mm_P10.16mm_Horizontal"
-			(at 111.252 123.19 90)
-			(effects
-				(font
-					(size 1.27 1.27)
-				)
-				(hide yes)
-			)
-		)
-		(property "Datasheet" "~"
-			(at 113.03 123.19 0)
-			(effects
-				(font
-					(size 1.27 1.27)
-				)
-				(hide yes)
-			)
-		)
-		(property "Description" "Resistor"
-			(at 113.03 123.19 0)
-			(effects
-				(font
-					(size 1.27 1.27)
-				)
-				(hide yes)
-			)
-		)
-		(pin "2"
-		)
-		(pin "1"
-		)
-		(instances
-			(project "board"
-				(path "/afefa398-9f39-4b22-97f8-dae9b102df0d/e2759770-a9ef-4fa2-921d-b35f031ff7ee"
-					(reference "R10")
-					(unit 1)
-				)

Commit message: capture ENGINE in schematic; fix couple of shorts
Parts:
- renumbered C4 to C2, C5 to C3, R13 to R10, R28 to R11, R17 to R12, R18 to R13, R29 to R14, R3 to R4, R4 to R5, R24 to R6, R8 to R7, R11 to R8, R27 to R9, U1 to U2
Connections:
- net FC0: no longer R9.2, U2.27 (FC1)
- net R/~{W}: no longer R8.2, U2.6 (~{AS})
- new net FC1: R9.2, U2.27 (FC1)
- new net ~{AS}: R8.2, U2.6 (~{AS})
Changed lines of the file:
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@@
 	)
 	(junction
-		(at 111.76 44.45)
-		(diameter 0)
-		(color 0 0 0 0)
-	)
-	(junction
 		(at 105.41 26.67)
 		(diameter 0)
@@
 	)
 	(junction
-		(at 107.95 97.79)
-		(diameter 0)
-		(color 0 0 0 0)
-	)
-	(junction
 		(at 105.41 44.45)
 		(diameter 0)
@@
 	(wire
 		(pts
-			(xy 107.95 97.79) (xy 143.51 97.79)
+			(xy 101.6 97.79) (xy 143.51 97.79)
 		)
 		(stroke
@@
 	(wire
 		(pts
-			(xy 111.76 44.45) (xy 143.51 44.45)
+			(xy 105.41 44.45) (xy 143.51 44.45)
 		)
 		(stroke
@@
 	(wire
 		(pts
-			(xy 101.6 97.79) (xy 107.95 97.79)
-		)
-		(stroke
-			(width 0)
-			(type default)
-		)
-	)
-	(wire
-		(pts
 			(xy 173.99 87.63) (xy 184.15 87.63)
 		)
@@
 	(wire
 		(pts
-			(xy 105.41 44.45) (xy 111.76 44.45)
-		)
-		(stroke
-			(width 0)
-			(type default)
-		)
-	)
-	(wire
-		(pts
 			(xy 173.99 85.09) (xy 184.15 85.09)
 		)
@@
 		(dnp no)
 		(fields_autoplaced yes)
-		(property "Reference" "#PWR076"
+		(property "Reference" "#PWR026"
 			(at 101.6 78.74 0)
 			(effects
@@
 			(project "board"
 				(path "/afefa398-9f39-4b22-97f8-dae9b102df0d/e2759770-a9ef-4fa2-921d-b35f031ff7ee"
-					(reference "#PWR076")
+					(reference "#PWR026")
 					(unit 1)
 				)
@@
 		(dnp no)
 		(fields_autoplaced yes)
-		(property "Reference" "#PWR020"
+		(property "Reference" "#PWR028"
 			(at 105.41 25.4 0)
 			(effects
@@
 			(project "board"
 				(path "/afefa398-9f39-4b22-97f8-dae9b102df0d/e2759770-a9ef-4fa2-921d-b35f031ff7ee"
-					(reference "#PWR020")
+					(reference "#PWR028")
 					(unit 1)
 				)
@@
 		(dnp no)
 		(fields_autoplaced yes)
-		(property "Reference" "#PWR019"
+		(property "Reference" "#PWR033"
 			(at 158.75 147.32 0)
 			(effects
@@
 			(project "board"
 				(path "/afefa398-9f39-4b22-97f8-dae9b102df0d/e2759770-a9ef-4fa2-921d-b35f031ff7ee"
-					(reference "#PWR019")
+					(reference "#PWR033")
 					(unit 1)
 				)
@@
 		(on_board yes)
 		(dnp no)
-		(property "Reference" "R4"
+		(property "Reference" "R5"
 			(at 87.122 54.61 0)
 			(effects
@@
 			(project "board"
 				(path "/afefa398-9f39-4b22-97f8-dae9b102df0d/e2759770-a9ef-4fa2-921d-b35f031ff7ee"
-					(reference "R4")
+					(reference "R5")
 					(unit 1)
 				)
@@
 		(on_board yes)
 		(dnp no)
-		(property "Reference" "#PWR077"
+		(property "Reference" "#PWR029"
 			(at 127 78.74 0)
 			(effects
@@
 			(project "board"
 				(path "/afefa398-9f39-4b22-97f8-dae9b102df0d/e2759770-a9ef-4fa2-921d-b35f031ff7ee"
-					(reference "#PWR077")
+					(reference "#PWR029")
 					(unit 1)
 				)
@@
 		(on_board yes)
 		(dnp no)
-		(property "Reference" "R18"
+		(property "Reference" "R13"
 			(at 118.872 39.37 0)
 			(effects
@@
 			(project "board"
 				(path "/afefa398-9f39-4b22-97f8-dae9b102df0d/e2759770-a9ef-4fa2-921d-b35f031ff7ee"
-					(reference "R18")
+					(reference "R13")
 					(unit 1)
 				)
@@
 		(dnp no)
 		(fields_autoplaced yes)
-		(property "Reference" "C5"
+		(property "Reference" "C3"
 			(at 156.21 154.9399 0)
 			(effects
@@
 			(project "board"
 				(path "/afefa398-9f39-4b22-97f8-dae9b102df0d/e2759770-a9ef-4fa2-921d-b35f031ff7ee"
-					(reference "C5")
+					(reference "C3")
 					(unit 1)
 				)
@@
 		(on_board yes)
 		(dnp no)
-		(property "Reference" "U1"
+		(property "Reference" "U2"
 			(at 160.8933 29.21 0)
 			(effects
@@
 			(project ""
 				(path "/afefa398-9f39-4b22-97f8-dae9b102df0d/e2759770-a9ef-4fa2-921d-b35f031ff7ee"
-					(reference "U1")
+					(reference "U2")
 					(unit 1)
 				)
@@
 		(dnp no)
 		(fields_autoplaced yes)
-		(property "Reference" "C4"
+		(property "Reference" "C2"
 			(at 140.97 154.9399 0)
 			(effects
@@
 			(project "board"
 				(path "/afefa398-9f39-4b22-97f8-dae9b102df0d/e2759770-a9ef-4fa2-921d-b35f031ff7ee"
-					(reference "C4")
+					(reference "C2")
 					(unit 1)
 				)
@@
 		(on_board yes)
 		(dnp no)
-		(property "Reference" "R28"
+		(property "Reference" "R11"
 			(at 108.712 86.36 0)
 			(effects
@@
 			(project "board"
 				(path "/afefa398-9f39-4b22-97f8-dae9b102df0d/e2759770-a9ef-4fa2-921d-b35f031ff7ee"
-					(reference "R28")
+					(reference "R11")
 					(unit 1)
 				)
@@
 		(on_board yes)
 		(dnp no)
-		(property "Reference" "R24"
+		(property "Reference" "R6"
 			(at 96.012 86.36 0)
 			(effects
@@
 			(project "board"
 				(path "/afefa398-9f39-4b22-97f8-dae9b102df0d/e2759770-a9ef-4fa2-921d-b35f031ff7ee"
-					(reference "R24")
+					(reference "R6")
 					(unit 1)
 				)
@@
 		(dnp no)
 		(fields_autoplaced yes)
-		(property "Reference" "#PWR017"
+		(property "Reference" "#PWR031"
 			(at 137.16 166.37 0)
 			(effects
@@
 			(project "board"
 				(path "/afefa398-9f39-4b22-97f8-dae9b102df0d/e2759770-a9ef-4fa2-921d-b35f031ff7ee"
-					(reference "#PWR017")
+					(reference "#PWR031")
 					(unit 1)
 				)
@@
 		(dnp no)
 		(fields_autoplaced yes)
-		(property "Reference" "R8"
+		(property "Reference" "R7"
 			(at 105.41 121.9199 0)
 			(effects
@@
 			(project "board"
 				(path "/afefa398-9f39-4b22-97f8-dae9b102df0d/e2759770-a9ef-4fa2-921d-b35f031ff7ee"
-					(reference "R8")
+					(reference "R7")
 					(unit 1)
 				)
@@
 		(dnp no)
 		(fields_autoplaced yes)
-		(property "Reference" "#PWR014"
+		(property "Reference" "#PWR025"
 			(at 85.09 46.99 0)
 			(effects
@@
 			(project "board"
 				(path "/afefa398-9f39-4b22-97f8-dae9b102df0d/e2759770-a9ef-4fa2-921d-b35f031ff7ee"
-					(reference "#PWR014")
+					(reference "#PWR025")
 					(unit 1)
 				)
@@
 		(on_board yes)
 		(dnp no)
-		(property "Reference" "R27"
+		(property "Reference" "R9"
 			(at 102.362 92.71 0)
 			(effects
@@
 			(project "board"
 				(path "/afefa398-9f39-4b22-97f8-dae9b102df0d/e2759770-a9ef-4fa2-921d-b35f031ff7ee"
-					(reference "R27")
+					(reference "R9")
 					(unit 1)
 				)
@@
 		(dnp no)
 		(fields_autoplaced yes)
-		(property "Reference" "#PWR016"
+		(property "Reference" "#PWR030"
 			(at 137.16 156.21 0)
 			(effects
@@
 			(project "board"
 				(path "/afefa398-9f39-4b22-97f8-dae9b102df0d/e2759770-a9ef-4fa2-921d-b35f031ff7ee"
-					(reference "#PWR016")
+					(reference "#PWR030")
 					(unit 1)
 				)
@@
 		(on_board yes)
 		(dnp no)
-		(property "Reference" "R3"
+		(property "Reference" "R4"
 			(at 79.502 48.26 0)
 			(effects
@@
 			(project ""
 				(path "/afefa398-9f39-4b22-97f8-dae9b102df0d/e2759770-a9ef-4fa2-921d-b35f031ff7ee"
-					(reference "R3")
+					(reference "R4")
 					(unit 1)
 				)
@@
 		(dnp no)
 		(fields_autoplaced yes)
-		(property "Reference" "R29"
+		(property "Reference" "R14"
 			(at 129.54 82.5499 0)
 			(effects
@@
 			(project "board"
 				(path "/afefa398-9f39-4b22-97f8-dae9b102df0d/e2759770-a9ef-4fa2-921d-b35f031ff7ee"
-					(reference "R29")
+					(reference "R14")
 					(unit 1)
 				)
@@
 		(on_board yes)
 		(dnp no)
-		(property "Reference" "#PWR018"
+		(property "Reference" "#PWR032"
 			(at 158.75 30.48 0)
 			(effects
@@
 			(project "board"
 				(path "/afefa398-9f39-4b22-97f8-dae9b102df0d/e2759770-a9ef-4fa2-921d-b35f031ff7ee"
-					(reference "#PWR018")
+					(reference "#PWR032")
 					(unit 1)
 				)
@@
 		(on_board yes)
 		(dnp no)
-		(property "Reference" "R11"
+		(property "Reference" "R8"
 			(at 99.822 33.02 0)
 			(effects
@@
 			(project "board"
 				(path "/afefa398-9f39-4b22-97f8-dae9b102df0d/e2759770-a9ef-4fa2-921d-b35f031ff7ee"
-					(reference "R11")
+					(reference "R8")
 					(unit 1)
 				)
@@
 		(on_board yes)
 		(dnp no)
-		(property "Reference" "R17"
+		(property "Reference" "R12"
 			(at 112.522 33.02 0)
 			(effects
@@
 			(project "board"
 				(path "/afefa398-9f39-4b22-97f8-dae9b102df0d/e2759770-a9ef-4fa2-921d-b35f031ff7ee"
-					(reference "R17")
+					(reference "R12")
 					(unit 1)
 				)
@@
 		(on_board yes)
 		(dnp no)
-		(property "Reference" "#PWR015"
+		(property "Reference" "#PWR027"
 			(at 102.87 118.11 0)
 			(effects
@@
 			(project "board"
 				(path "/afefa398-9f39-4b22-97f8-dae9b102df0d/e2759770-a9ef-4fa2-921d-b35f031ff7ee"
-					(reference "#PWR015")
+					(reference "#PWR027")
 					(unit 1)
 				)
@@
 		(on_board yes)
 		(dnp no)
-		(property "Reference" "R13"
+		(property "Reference" "R10"
 			(at 106.172 39.37 0)
 			(effects
@@
 			(project "board"
 				(path "/afefa398-9f39-4b22-97f8-dae9b102df0d/e2759770-a9ef-4fa2-921d-b35f031ff7ee"
-					(reference "R13")
+					(reference "R10")
 					(unit 1)
 				)
