File: board/ram.kicad_sch (KiCad schematic)
At the start: 16 parts, among them U10 RAM 4 LO, U11 RAM 4 HI, U4 RAM 1 LO, U5 RAM 1 HI, U6 RAM 2 LO, U7 RAM 2 HI, U8 RAM 3 LO, U9 RAM 3 HI

Commit message: capture ENGINE in schematic; fix couple of shorts
Parts:
- renumbered C12 to C10, C13 to C11, C14 to C12, C15 to C13, C8 to C6, C9 to C7, C10 to C8, C11 to C9, U9 to U10, U10 to U11, U11 to U12, U4 to U5, U5 to U6, U6 to U7, U7 to U8, U8 to U9
