File: board/pixel.kicad_sch (KiCad schematic)
At the start: 8 parts, among them U20 PIXEL, U22 IDT7200L15P, U23 IDT7200L15P

Commit message: add VIDCMD FIFOs; FIFO strobe termination becomes a 0R-stuffed footprint
Co-Authored-By: Claude Fable 5.1 <noreply@anthropic.com>
Claude-Session: https://claude.ai/code/session_01NsFH8WNb3Tja14xUfwuyqj
Parts:
- R28, R29: value 47R -> 0R
Changed lines of the file:
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@@
 			)
 		)
-		(property "Value" "47R"
+		(property "Value" "0R"
 			(at 234.95 110.744 90)
 			(effects
@@
 			)
 		)
-		(property "Value" "47R"
+		(property "Value" "0R"
 			(at 234.95 37.084 90)
 			(effects
