File: board/audio-fifo.kicad_sch (KiCad schematic)
At the start: 5 parts

Commit message: add DEBUG_HEADER sheet (2x16 LogicAnalyzer V2 pinout); re-annotate AUDIO_FIFO
Co-Authored-By: Claude Fable 5.1 <noreply@anthropic.com>
Claude-Session: https://claude.ai/code/session_01NsFH8WNb3Tja14xUfwuyqj
Parts:
- removed C? (x2): 100nF, Capacitor_THT:C_Disc_D5.0mm_W2.5mm_P5.00mm, symbol Device:C
- removed R?: 0R, Resistor_THT:R_Axial_DIN0207_L6.3mm_D2.5mm_P10.16mm_Horizontal, symbol Device:R
- removed U? (x2): IDT7200L15P, Package_DIP:DIP-28_W7.62mm, symbol Memory_RAM:IDT7201
- added C33, C34: 100nF, Capacitor_THT:C_Disc_D5.0mm_W2.5mm_P5.00mm, symbol Device:C
- added R31: 0R, Resistor_THT:R_Axial_DIN0207_L6.3mm_D2.5mm_P10.16mm_Horizontal, symbol Device:R
- added U26, U27: IDT7200L15P, Package_DIP:DIP-28_W7.62mm, symbol Memory_RAM:IDT7201
Connections:
- net +5V: now also C33.1, C34.1, U26.23 (FL), U26.28 (VCC), U27.23 (FL), U27.28 (VCC)
- net AUDIO_L0: now also U26.9 (Q0)
- net AUDIO_L1: now also U26.10 (Q1)
- net AUDIO_L2: now also U26.11 (Q2)
- net AUDIO_L3: now also U26.12 (Q3)
- net AUDIO_L4: now also U26.16 (Q4)
- net AUDIO_L5: now also U26.17 (Q5)
- net AUDIO_L6: now also U26.18 (Q6)
- net AUDIO_L7: now also U26.19 (Q7)
- net AUDIO_R0: now also U27.9 (Q0)
- net AUDIO_R1: now also U27.10 (Q1)
- net AUDIO_R2: now also U27.11 (Q2)
- net AUDIO_R3: now also U27.12 (Q3)
- net AUDIO_R4: now also U27.16 (Q4)
- net AUDIO_R5: now also U27.17 (Q5)
- net AUDIO_R6: now also U27.18 (Q6)
- net AUDIO_R7: now also U27.19 (Q7)
- net D0: now also U27.6 (D0)
- net D1: now also U27.5 (D1)
- net D10: now also U26.4 (D2)
- net D11: now also U26.3 (D3)
- net D12: now also U26.27 (D4)
- net D13: now also U26.26 (D5)
- net D14: now also U26.25 (D6)
- net D15: now also U26.24 (D7)
- net D2: now also U27.4 (D2)
- net D3: now also U27.3 (D3)
- net D4: now also U27.27 (D4)
- net D5: now also U27.26 (D5)
- net D6: now also U27.25 (D6)
- net D7: now also U27.24 (D7)
- net D8: now also U26.6 (D0)
- net D9: now also U26.5 (D1)
- net GND: now also C33.2, C34.2, U26.14 (VSS), U26.2 (D8), U26.7 (XI), U27.14 (VSS), U27.2 (D8), U27.7 (XI)
- net ~{AUDIO_FIFO_EF}: now also U27.21 (EF)
- net ~{AUDIO_FIFO_RE_FIFO_SIDE}: now also R31.2, U26.15 (RD), U27.15 (RD)
- net ~{AUDIO_FIFO_RE}: now also R31.1
- net ~{AUDIO_FIFO_RS}: now also U26.22 (CLR), U27.22 (CLR)
- net ~{AUDIO_FIFO_W}: now also U26.1 (WR), U27.1 (WR)
