File: board/audio-fifo.kicad_sch (KiCad schematic)
At the start: 5 parts, among them U26 IDT7200L15P, U27 IDT7200L15P

Commit message: add debug header
Parts:
- renumbered C34 to C?, C33 to C?, R31 to R?, U26 to U?, U27 to U?
