File: board/debug-header.kicad_sch (KiCad schematic)
At the start: 3 parts, among them J8 DEBUG_HEADER, J9 DEBUG_HEADER

Commit message: add debug header
Parts:
- renumbered J8 to J?, J9 to J?, R32 to R?
